File: Hardware/292/292-power/292-power.kicad_sch (KiCad schematic)
At the start: 4 parts

Commit message: Draft board design
Parts:
- removed U?: T-USB_Expander_FR2032IG56, Package_SO:HTSSOP-56-1EP_6.1x14mm_P0.5mm_EP3.61x6.35mm, symbol Ziloo:T-USB_Expander_FR2032IG56
- removed U?: TCA9534PWR, Ziloo:TCA9534PWR, symbol Ziloo:TCA9534PWR
- added P2: PW, Ziloo:HRS_DF40C-50DS-0.4V(51), symbol Ziloo:292_PWRCTL-50
- added R1: R, Resistor_SMD:R_0402_1005Metric, symbol Device:R
- added U1: W25X40CLSN, Package_SO:SOIC-8_3.9x4.9mm_P1.27mm, symbol Memory_Flash:W25X40CLSN
- P1: renamed from P?; value T-USB_HIGH-SPEED-50 -> HS; symbol Ziloo:T-USB_HIGH-SPEED-50 -> Ziloo:292_HIGH-SPEED-50
- U2: renamed from U?; footprint RSH0056E -> Ziloo:TPS65988DHRSHR
Connections:
- net BAT_CE: now also U2.49 (GPIO17_PP_EXT2), P2.24 (BAT_CE#)
- net BAT_INT: now also U2.48 (GPIO16_PP_EXT1), P2.23 (BAT_INT)
- net BAT_STAT: now also P2.22 (BAT_STAT); no longer P1.25 (BAT_STAT)
- net GND: now also P1.33 (GND), P2.11 (GND), P2.2 (GND), P2.5 (GND), P2.8 (GND), U1.4 (GND)
- net POWER_SCL: now also U2.21 (I2C3_SCL_GPIO5), P2.36 (POWER_SCL)
- net POWER_SDA: now also U2.22 (I2C3_SDA_GPIO6), P2.35 (POWER_SDA)
- net PWR_CHARGE: now also P1.30 (PWR_CHARGE); no longer P1.24 (PWR_CHARGE)
- net STEM SCL: now also P1.17 (STEM_SCL), U2.27 (I2C1_SCL)
- net STEM SDA: now also P1.18 (STEM_SDA), U2.28 (I2C1_SDA)
- net SYS SCL: now also U2.32 (I2C2_SCL), P2.13 (SYS_I2C_SCL)
- net SYS SDA: now also U2.33 (I2C2_SDA), P2.14 (SYS_I2C_SDA)
- net USB_XD_OE: now reaches U2.17 (GPIO1)
- net USB_XD_OE: now also P2.16 (USB_XD_OE)
- net USB_XD_SEL: now reaches U2.18 (GPIO2)
- net USB_XD_SEL: now also P2.17 (USB_XD_SEL)
- net POWER_PD_CTL_INT: now reaches U2.23 (I2C3_IRQ_GPIO7_N)
- net POWER_PD_CTL_INT: now also P2.37 (POWER_PD_CTL_INT)
- net OTG_CC1: now reaches U2.24 (C1_CC1)
- net OTG_CC2: now reaches U2.26 (C1_CC2)
- net at U2.29 (I2C1_IRQ_N): now also P1.19 (STEM_INT)
- net OTG_2.0_FAULT: now reaches U2.30 (HPD1_GPIO3)
- net HOST_HPD_RSVD: now reaches U2.31 (HPD2_GPIO4)
- net SYS_PD_CTL_INT: now reaches U2.34 (I2C2_IRQ_N)
- net SYS_PD_CTL_INT: now also P2.12 (SYS_PD_CTL_INT)
- net SPI_MISO: now reaches U2.36 (SPI_MISO_GPIO8)
- net SPI_MISO: now also P2.31 (SPI_MISO), U1.2 (DO(IO1))
- net SPI_MOSI: now reaches U2.37 (SPI_MOSI_GPIO9)
- net SPI_MOSI: now also P2.30 (SPI_MOSI), U1.5 (DI(IO0))
- net SPI_CLK: now reaches U2.38 (SPI_CLK_GPIO10)
- net SPI_CLK: now also P2.32 (SPI_CLK), U1.6 (SCK)
- net SPI_SS: now reaches U2.39 (SPI_SS_GPIO11_N)
- net SPI_SS: now also P2.33 (SPI_CS), U1.1 (~{CS})
- net BAT_EN: now reaches U2.40 (GPIO12)
- net BAT_EN: now also P2.25 (BAT_EN)
- net LOCK_BTN: now reaches U2.41 (GPIO13)
- net LOCK_BTN: now also P2.28 (LOCK_BTN)
- net PD_HRESET: now reaches U2.44 (HRESET)
- net PD_HRESET: now also P2.39 (PD_HRESET)
- net OTG_D+: now reaches U2.50 (C1_USB_P_GPIO18)
- net OTG_D+: now also P2.3 (USB1_DP)
- net OTG_D-: now reaches U2.53 (C1_USB_N_GPIO19)
- net OTG_D-: now also P2.4 (USB1_DN)
- net HOST_D+: now reaches U2.54 (C2_USB_P_GPIO20)
- net HOST_D+: now also P2.6 (USB2_DP)
- net HOST_D-: now reaches U2.55 (C2_USB_N_GPIO21)
- net HOST_D-: now also P2.7 (USB2_DN)
- net VSOM: now reaches P1.1 (VSOM)
- net VSOM: now also P1.26 (VSOM), P1.36 (VSOM), P1.39 (VSOM), P1.42 (VSOM), P1.45 (VSOM), P1.48 (VSOM), P2.1 (VSOM), P2.15 (VSOM), P2.26 (VSOM)
- net T_SBWTCK: no longer names the net of P1.21
- net T_SBWTDIO: no longer names the net of P1.23
- net UART_T_RXD: no longer names the net of P1.27
- net UART_T_TXD: no longer names the net of P1.28
- new net: R1.2, U1.3 (~{WP})
- new net BAT_3V3: P2.40 (3V3), P2.43 (3V3)
- new net BAT_5V: P2.46 (5V)
- new net BAT_LDO: P2.29 (BAT_LDO)
- new net FLASH_HOLD: P2.34 (FLASH_HOLD), U1.7 (~{HOLD})
- new net HOST_XD+: P2.45 (USB2_XDP)
- new net HOST_XD-: P2.44 (USB2_XDN)
- new net OTG_XD+: P2.48 (USB1_XDP)
- new net OTG_XD-: P2.47 (USB1_XDN)
- new net PD_LDO_3V3: R1.1, U1.8 (VCC)
- new net SHUTDOWN_BTN: P2.27 (SHUTDOWN_BTN)
- new net USB1_PLUG_INT: P2.38 (USB1_PLUG_INT)
- new net USB1_SBU1: P2.9 (USB1_SBU1)
- new net USB1_SBU2: P2.10 (USB1_SBU2)
- new net VCC_RTC: P2.49 (VCC_RTC)
- no-connect marks 12 -> 24
Other:
- added sheet OTG USB-C Connector (otg-usb-c.kicad_sch)
- note added: "Low during boot"
- note added: "Stem address 0x38 Power address 0x3F"
- note removed: "3.3V supplied whenever possible from PD Controller?"
- title: (none) -> 292 T-USB Power
- moved on the sheet: U2A

Commit message: Clarifications for the board plan
Connections:
- net USB1_PLUG_INT: no longer names the net of P2.38 (USB1_PLUG_INT)
- no-connect marks 24 -> 25
Changed lines of the file:
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@@
   (junction (at 196.85 139.7) (diameter 0) (color 0 0 0 0)
   )
+  (no_connect (at 261.62 134.62))
   (no_connect (at 261.62 104.14))
   (no_connect (at 223.52 262.89))
@@
     (stroke (width 0) (type default) (color 0 0 0 0))
   )
-  (wire (pts (xy 205.74 97.79) (xy 172.72 97.79))
-    (stroke (width 0) (type default) (color 0 0 0 0))
-  )
   (wire (pts (xy 67.31 306.07) (xy 82.55 306.07))
     (stroke (width 0) (type default) (color 0 0 0 0))
@@
     (stroke (width 0) (type default) (color 0 0 0 0))
   )
+  (wire (pts (xy 101.6 207.01) (xy 124.46 207.01))
+    (stroke (width 0) (type default) (color 0 0 0 0))
+  )
   (wire (pts (xy 36.83 260.35) (xy 45.72 260.35))
     (stroke (width 0) (type default) (color 0 0 0 0))
@@
     (stroke (width 0) (type default) (color 0 0 0 0))
   )
-  (wire (pts (xy 261.62 134.62) (xy 281.94 134.62))
-    (stroke (width 0) (type default) (color 0 0 0 0))
-  )
   (wire (pts (xy 261.62 157.48) (xy 276.86 157.48))
     (stroke (width 0) (type default) (color 0 0 0 0))
@@
     (stroke (width 0) (type default) (color 0 0 0 0))
   )
-  (wire (pts (xy 281.94 134.62) (xy 281.94 88.9))
-    (stroke (width 0) (type default) (color 0 0 0 0))
-  )
   (wire (pts (xy 104.14 165.1) (xy 123.19 165.1))
     (stroke (width 0) (type default) (color 0 0 0 0))
@@
     (stroke (width 0) (type default) (color 0 0 0 0))
   )
-  (wire (pts (xy 281.94 88.9) (xy 205.74 88.9))
-    (stroke (width 0) (type default) (color 0 0 0 0))
-  )
   (wire (pts (xy 205.74 207.01) (xy 205.74 109.22))
     (stroke (width 0) (type default) (color 0 0 0 0))
@@
     (stroke (width 0) (type default) (color 0 0 0 0))
   )
-  (wire (pts (xy 205.74 88.9) (xy 205.74 97.79))
-    (stroke (width 0) (type default) (color 0 0 0 0))
-  )
   (wire (pts (xy 191.77 102.87) (xy 191.77 144.78))
     (stroke (width 0) (type default) (color 0 0 0 0))
@@
     (effects (font (size 1.27 1.27)) (justify left bottom))
   )
+  (label "OTG_D-" (at 173.99 123.19 0)
+    (effects (font (size 1.27 1.27)) (justify left bottom))
+  )
   (label "POWER SDA" (at 265.43 142.24 0)
     (effects (font (size 1.27 1.27)) (justify left bottom))
@@
     (effects (font (size 1.27 1.27)) (justify left bottom))
   )
-  (label "USB1_PLUG_INT" (at 265.43 88.9 0)
-    (effects (font (size 1.27 1.27)) (justify left bottom))
-  )
   (label "USB_XD_SEL" (at 215.9 144.78 0)
     (effects (font (size 1.27 1.27)) (justify left bottom))
@@
     (effects (font (size 1.27 1.27)) (justify left bottom))
   )
+  (label "POWER_PD_CTL_INT" (at 104.14 207.01 0)
+    (effects (font (size 1.27 1.27)) (justify left bottom))
+  )
+  (label "OTG_D+" (at 173.99 120.65 0)
+    (effects (font (size 1.27 1.27)) (justify left bottom))
+  )
   (label "SPI_CLK" (at 265.43 149.86 0)
     (effects (font (size 1.27 1.27)) (justify left bottom))
@@
     (effects (font (size 1.27 1.27)) (justify right))
   )
+  (hierarchical_label "POWER_PD_CTL_INT" (shape input) (at 124.46 207.01 0)
+    (effects (font (size 1.27 1.27)) (justify left))
+  )
   (hierarchical_label "USB_XD_OE" (shape input) (at 170.18 210.82 180)
     (effects (font (size 1.27 1.27)) (justify right))
@@
   )
   (hierarchical_label "USB_XD_SEL" (shape input) (at 170.18 213.36 180)
-    (effects (font (size 1.27 1.27)) (justify right))
-  )
-  (hierarchical_label "USB1_PLUG_INT" (shape input) (at 172.72 97.79 180)
     (effects (font (size 1.27 1.27)) (justify right))
   )
@@
       (reference "D2") (unit 1) (value "D_Schottky") (footprint "Diode_SMD:D_0402_1005Metric")
     )
+    (path "/004f8629-4657-48c8-b70f-4d83fd7acfae/91eb054e-468a-4ebd-955a-9a5c84ba8a31"
+      (reference "D?") (unit 1) (value "LED") (footprint "")
+    )
     (path "/004f8629-4657-48c8-b70f-4d83fd7acfae/050a1568-eb0f-40c9-89a6-50f798528697"
       (reference "J1") (unit 1) (value "Lock") (footprint "Connector_JST:JST_ACH_BM03B-ACHSS-GAN-ETF_1x03-1MP_P1.20mm_Vertical")
@@
     )
     (path "/004f8629-4657-48c8-b70f-4d83fd7acfae/b1064037-54eb-4ee0-be21-3fd44471f7d4"
-      (reference "L1") (unit 1) (value "L") (footprint "Inductor_SMD:L_0805_2012Metric")
+      (reference "L1") (unit 1) (value "1.0uH") (footprint "Inductor_SMD:L_0805_2012Metric")
     )
     (path "/7c602596-028d-4f8d-ab90-830f025a564d"
@@
       (reference "R32") (unit 1) (value "10K") (footprint "Resistor_SMD:R_0402_1005Metric")
     )
+    (path "/004f8629-4657-48c8-b70f-4d83fd7acfae/4e8d3dae-a8b7-4768-8e19-8da4ba404b67"
+      (reference "R?") (unit 1) (value "R") (footprint "Resistor_SMD:R_0402_1005Metric")
+    )
     (path "/aeb3a014-4174-4720-9923-dafc56899db9"

Commit message: First review based revision
Connections:
- net GND: now also P1.16, P1.23
- net BAT_3V3 renamed LIVE_3V3
- net BAT_5V renamed LIVE_5V
- no-connect marks 25 -> 24
Changed lines of the file:
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@@
   (junction (at 260.35 237.49) (diameter 0) (color 0 0 0 0)
+  )
+  (junction (at 219.71 240.03) (diameter 0) (color 0 0 0 0)
+  )
+  (junction (at 219.71 257.81) (diameter 0) (color 0 0 0 0)
   )
   (junction (at 196.85 139.7) (diameter 0) (color 0 0 0 0)
@@
   (no_connect (at 223.52 255.27))
   (no_connect (at 223.52 252.73))
-  (no_connect (at 223.52 257.81))
   (no_connect (at 261.62 124.46))
   (no_connect (at 261.62 127))
@@
     (stroke (width 0) (type default) (color 0 0 0 0))
   )
+  (wire (pts (xy 219.71 240.03) (xy 219.71 250.19))
+    (stroke (width 0) (type default) (color 0 0 0 0))
+  )
   (wire (pts (xy 177.8 267.97) (xy 177.8 247.65))
     (stroke (width 0) (type default) (color 0 0 0 0))
@@
     (stroke (width 0) (type default) (color 0 0 0 0))
   )
-  (wire (pts (xy 219.71 232.41) (xy 219.71 250.19))
+  (wire (pts (xy 219.71 232.41) (xy 219.71 240.03))
     (stroke (width 0) (type default) (color 0 0 0 0))
   )
@@
     (stroke (width 0) (type default) (color 0 0 0 0))
   )
-  (wire (pts (xy 101.6 110.49) (xy 127 110.49))
-    (stroke (width 0) (type default) (color 0 0 0 0))
-  )
   (wire (pts (xy 67.31 300.99) (xy 82.55 300.99))
     (stroke (width 0) (type default) (color 0 0 0 0))
@@
     (stroke (width 0) (type default) (color 0 0 0 0))
   )
+  (wire (pts (xy 219.71 257.81) (xy 223.52 257.81))
+    (stroke (width 0) (type default) (color 0 0 0 0))
+  )
   (wire (pts (xy 261.62 144.78) (xy 273.05 144.78))
     (stroke (width 0) (type default) (color 0 0 0 0))
@@
     (stroke (width 0) (type default) (color 0 0 0 0))
   )
+  (wire (pts (xy 111.76 160.02) (xy 123.19 160.02))
+    (stroke (width 0) (type default) (color 0 0 0 0))
+  )
+  (wire (pts (xy 219.71 257.81) (xy 219.71 269.24))
+    (stroke (width 0) (type default) (color 0 0 0 0))
+  )
   (wire (pts (xy 172.72 242.57) (xy 172.72 262.89))
     (stroke (width 0) (type default) (color 0 0 0 0))
@@
     (stroke (width 0) (type default) (color 0 0 0 0))
   )
-  (wire (pts (xy 101.6 160.02) (xy 101.6 110.49))
-    (stroke (width 0) (type default) (color 0 0 0 0))
-  )
   (wire (pts (xy 194.31 142.24) (xy 194.31 100.33))
     (stroke (width 0) (type default) (color 0 0 0 0))
@@
     (stroke (width 0) (type default) (color 0 0 0 0))
   )
-  (wire (pts (xy 219.71 250.19) (xy 219.71 269.24))
+  (wire (pts (xy 219.71 250.19) (xy 219.71 257.81))
     (stroke (width 0) (type default) (color 0 0 0 0))
   )
@@
     (stroke (width 0) (type default) (color 0 0 0 0))
   )
-  (wire (pts (xy 101.6 160.02) (xy 123.19 160.02))
-    (stroke (width 0) (type default) (color 0 0 0 0))
-  )
   (wire (pts (xy 227.33 91.44) (xy 229.87 91.44))
     (stroke (width 0) (type default) (color 0 0 0 0))
@@
     (stroke (width 0) (type default) (color 0 0 0 0))
   )
+  (wire (pts (xy 219.71 240.03) (xy 223.52 240.03))
+    (stroke (width 0) (type default) (color 0 0 0 0))
+  )
   (wire (pts (xy 191.77 102.87) (xy 191.77 144.78))
     (stroke (width 0) (type default) (color 0 0 0 0))
@@
     (effects (font (size 1.27 1.27)) (justify left bottom))
   )
-  (label "BAT_3V3" (at 264.16 121.92 0)
+  (label "LIVE_3V3" (at 264.16 121.92 0)
     (effects (font (size 1.27 1.27)) (justify left bottom))
   )
@@
     (effects (font (size 1.27 1.27)) (justify left bottom))
   )
-  (label "BAT_3V3" (at 113.03 157.48 0)
+  (label "LIVE_3V3" (at 113.03 157.48 0)
     (effects (font (size 1.27 1.27)) (justify left bottom))
   )
@@
     (effects (font (size 1.27 1.27)) (justify left bottom))
   )
+  (label "OTG_2.0_FAULT" (at 67.31 252.73 0)
+    (effects (font (size 1.27 1.27)) (justify left bottom))
+  )
   (label "SYS SDA" (at 218.44 137.16 0)
     (effects (font (size 1.27 1.27)) (justify left bottom))
@@
     (effects (font (size 1.27 1.27)) (justify left bottom))
   )
-  (label "BAT_5V" (at 113.03 160.02 0)
+  (label "LIVE_5V" (at 113.03 160.02 0)
     (effects (font (size 1.27 1.27)) (justify left bottom))
   )
@@
     (effects (font (size 1.27 1.27)) (justify left bottom))
   )
-  (label "BAT_5V" (at 264.16 114.3 0)
+  (label "LIVE_5V" (at 264.16 114.3 0)
     (effects (font (size 1.27 1.27)) (justify left bottom))
   )
@@
     (effects (font (size 1.27 1.27)) (justify left bottom))
   )
-  (label "BAT_3V3" (at 264.16 129.54 0)
+  (label "LIVE_3V3" (at 264.16 129.54 0)
     (effects (font (size 1.27 1.27)) (justify left bottom))
   )
@@
     (effects (font (size 1.27 1.27)) (justify right))
   )
-  (hierarchical_label "VIN_3V3" (shape input) (at 127 107.95 0)
+  (hierarchical_label "LIVE_3V3" (shape input) (at 127 107.95 0)
     (effects (font (size 1.27 1.27)) (justify left))
   )
@@
     (effects (font (size 1.27 1.27)) (justify right))
   )
-  (hierarchical_label "BAT_5V" (shape input) (at 123.19 160.02 0)
+  (hierarchical_label "LIVE_5V" (shape input) (at 123.19 160.02 0)
     (effects (font (size 1.27 1.27)) (justify left))
   )
@@
     (effects (font (size 1.27 1.27)) (justify right))
   )
-  (hierarchical_label "VIN_3V3" (shape input) (at 124.46 209.55 0)
+  (hierarchical_label "LIVE_3V3" (shape input) (at 124.46 209.55 0)
     (effects (font (size 1.27 1.27)) (justify left))
   )
@@
     (effects (font (size 1.27 1.27)) (justify right))
   )
-  (hierarchical_label "VIN_5V" (shape input) (at 127 110.49 0)
-    (effects (font (size 1.27 1.27)) (justify left))
-  )
   (hierarchical_label "PD_LDO_1V8" (shape input) (at 123.19 147.32 0)
     (effects (font (size 1.27 1.27)) (justify left))
@@
     (effects (font (size 1.27 1.27)) (justify left))
   )
-  (hierarchical_label "BAT_3V3" (shape input) (at 123.19 157.48 0)
+  (hierarchical_label "LIVE_3V3" (shape input) (at 123.19 157.48 0)
     (effects (font (size 1.27 1.27)) (justify left))
   )
@@
       (reference "#PWR031") (unit 1) (value "GND") (footprint "")
     )
-    (path "/004f8629-4657-48c8-b70f-4d83fd7acfae/98b69f95-94e2-489d-8c54-fcf72279ab95"
-      (reference "#PWR0101") (unit 1) (value "GND") (footprint "")
-    )
     (path "/55bbf0fb-a337-4d8d-b52e-a8f2b654da48/aa7cd74b-4a7c-4b77-8981-4dde8ad03cfa"
       (reference "#PWR0103") (unit 1) (value "GND") (footprint "")
@@
       (reference "#PWR0106") (unit 1) (value "GND") (footprint "")
     )
+    (path "/004f8629-4657-48c8-b70f-4d83fd7acfae/2fb2e67e-2079-46b2-a4f5-89b8e25f424b"
+      (reference "#PWR?") (unit 1) (value "GND") (footprint "")
+    )
+    (path "/004f8629-4657-48c8-b70f-4d83fd7acfae/ab2b76bb-216f-4043-b114-8e8d2de2e8c1"
+      (reference "#PWR?") (unit 1) (value "GND") (footprint "")
+    )
+    (path "/004f8629-4657-48c8-b70f-4d83fd7acfae/bae0637d-141a-4a57-a4d0-65c617216942"
+      (reference "#PWR?") (unit 1) (value "GND") (footprint "")
+    )
+    (path "/004f8629-4657-48c8-b70f-4d83fd7acfae/cda05f16-d324-4125-9a70-59ddbb3365e9"
+      (reference "#PWR?") (unit 1) (value "GND") (footprint "")
+    )
     (path "/004f8629-4657-48c8-b70f-4d83fd7acfae/d2c63a70-73d4-4698-badf-4e2f0c273887"
       (reference "C1") (unit 1) (value "22uF") (footprint "Capacitor_SMD:C_0402_1005Metric")
@@
       (reference "C19") (unit 1) (value "0.1uF") (footprint "Capacitor_SMD:C_0402_1005Metric")
     )
+    (path "/004f8629-4657-48c8-b70f-4d83fd7acfae/18fb26fe-9492-4b47-80b6-991431a199d8"
+      (reference "C?") (unit 1) (value "C") (footprint "Capacitor_SMD:C_0402_1005Metric")
+    )
+    (path "/004f8629-4657-48c8-b70f-4d83fd7acfae/5cbf3823-f3cc-4684-8965-28d3411ca9fa"
+      (reference "C?") (unit 1) (value "5uF") (footprint "Capacitor_SMD:C_0402_1005Metric")
+    )
+    (path "/004f8629-4657-48c8-b70f-4d83fd7acfae/defb7e3a-760d-4402-9463-74fd540ca077"
+      (reference "C?") (unit 1) (value "C") (footprint "Capacitor_SMD:C_0402_1005Metric")
+    )
     (path "/004f8629-4657-48c8-b70f-4d83fd7acfae/59d643ee-2269-4a2a-a18e-827283db6342"
       (reference "D1") (unit 1) (value "D_Schottky") (footprint "Diode_SMD:D_0402_1005Metric")
@@
       (reference "U9") (unit 2) (value "TPD6S300ARUKR") (footprint "Ziloo:TPD6S300ARUKR")
     )
-  )
+    (path "/004f8629-4657-48c8-b70f-4d83fd7acfae/87d65e6b-c7bd-41c1-880c-46144b2b318c"
+      (reference "U?") (unit 1) (value "TPS79633DCQR") (footprint "Ziloo:TPS79618DCQR")
+    )
+    (path "/004f8629-4657-48c8-b70f-4d83fd7acfae/d4a1ca0d-df8e-46ec-81d0-8ab7850ba91a"
+      (reference "U?") (unit 1) (value "TPS79633DCQR") (footprint "Ziloo:TPS79618DCQR")
+    )
+  )
