File: Hardware/292/292-power/host-usb-c.kicad_sch (KiCad schematic)
At the start: 17 parts

Commit message: Draft board design
Parts:
- added R10, R11, R12, R13, R14, R15, R17, R18: 10K, Resistor_SMD:R_0402_1005Metric, symbol Device:R
- added U4: TS5USBC410YFFR, Ziloo:TS5USBC410YFFR, symbol Ziloo:TS5USBC410YFFR
- C10, C11, C12, C13, C8, C9: renamed from C?; footprint (none) -> Capacitor_SMD:C_0402_1005Metric
- J3: renamed from J?; value TUSB_C_Host_Receptacle -> Host; footprint (none) -> Ziloo:HIROSE_CX80B1-24P
- J4: renamed from J?; value T-USB-ALT-HOST_45_pins -> ALT-HOST; footprint Package_SO:TSSOP-24_4.4x7.8mm_P0.65mm -> Ziloo:4-2328724-5; symbol Ziloo:T-USB-ALT-HOST_45_pins -> Ziloo:292-ALT-HOST_45_pins
- R16, R19, R7, R8, R9: renamed from R?; footprint (none) -> Resistor_SMD:R_0402_1005Metric
- U6: renamed from U?; footprint WQFN20_RUK_TEX -> Ziloo:TPD6S300ARUKR
- gave numbers to parts that had none: 2
Connections:
- net GND: now also J4.16 (GND), J4.19 (GND), J4.24 (GND), J4.27 (GND), J4.30 (GND), J4.33 (GND), J4.36 (GND), J4.39 (GND), R11.2, R13.2, R15.2, R18.2, U4.B3 (GND)
- net LDO_3V3: no longer C12.1, C13.1, J4.1 (3V3), J4.10 (3V3), J4.13 (3V3), J4.4 (3V3), J4.7 (3V3), R16.1, R7.1, U5.1 (VCC), U5.20 (VCC), U5.28 (VCC), U5.6 (VCC), U6.10 (VPWER)
- net POWER_SCL: now also J4.40 (POWER_SCL)
- net POWER_SDA: now also J4.41 (POWER_SDA)
- net SBU1: now also U5.27 (SBU1)
- net SBU2: now also U5.26 (SBU2)
- net OTG_XD+: now reaches J4.20 (HX+)
- net OTG_XD+: now also U4.C1 (D2+)
- net OTG_XD-: now reaches J4.21 (HX-)
- net OTG_XD-: now also U4.C2 (D2-)
- net HOST_D+: now reaches J3.A6 (D+), U6.19 (D2)
- net HOST_D+: now also U4.C3 (D1+)
- net HOST_D-: now reaches J3.A7 (D-), U6.20 (D1)
- net HOST_D-: now also U4.C4 (D1-)
- net DPEQ1: now reaches U5.2 (DPEQ1)
- net DPEQ1: now also R10.2, R11.1
- net SSEQ1: now reaches U5.3 (SSEQ1)
- net SSEQ1: now also R12.2, R13.1
- net EQ1: now reaches U5.35 (EQ1)
- net EQ1: now also R17.2, R18.1
- net EQ0: now reaches U5.38 (EQ0)
- net EQ0: now also R14.2, R15.1
- net at J3.B6 (D+): now also U4.A2 (D+)
- net at J3.B7 (D-): now also U4.A3 (D-)
- net VBUS renamed HOST_VBUS
- new net OTG_2.0_FAULT: U4.A4 (FLT)
- new net USB_DX_OE: U4.B4 (OE)
- new net USB_DX_SEL: U4.A1 (SEL1), U4.B2 (SEL2)
- new net VIN_3V3: C12.1, C13.1, J4.1 (3V3), J4.10 (3V3), J4.13 (3V3), J4.4 (3V3), J4.7 (3V3), R10.1, R12.1, R14.1, R16.1, R17.1, R7.1, U4.B1 (VCC), U5.1 (VCC), U5.20 (VCC), U5.28 (VCC), U5.6 (VCC), U6.10 (VPWER)
- no-connect marks 1 -> 15
Other:
- note added: "Connects to - Keyboards - Mouse - Monitor"
- note removed: "HPDIN needs to be connected"
- note removed: "Should I2C3 of the TPS65 be able to control POWER I2C?"
- moved on the sheet: C10, C11, C12, C13, C8, C9, J3, J4, R16, R19, R7, R8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

Commit message: Clarifications for the board plan
Connections:
- net POWER_PD_CTL_INT: now reaches J4.42 (POWER_INT)
- no-connect marks 15 -> 18
Changed lines of the file:
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@@
   (no_connect (at 157.48 173.99))
   (no_connect (at 157.48 199.39))
+  (no_connect (at 44.45 266.7))
+  (no_connect (at 44.45 269.24))
+  (no_connect (at 44.45 264.16))
   (no_connect (at 83.82 219.71))
   (no_connect (at 44.45 220.98))
@@
     (stroke (width 0) (type default) (color 0 0 0 0))
   )
+  (wire (pts (xy 44.45 261.62) (xy 52.07 261.62))
+    (stroke (width 0) (type default) (color 0 0 0 0))
+  )
   (wire (pts (xy 144.78 184.15) (xy 175.26 184.15))
     (stroke (width 0) (type default) (color 0 0 0 0))
@@
     (effects (font (size 1.27 1.27)) (justify left))
   )
+  (hierarchical_label "POWER_PD_CTL_INT" (shape input) (at 52.07 261.62 0)
+    (effects (font (size 1.27 1.27)) (justify left))
+  )

Commit message: First review based revision
Connections:
- net OTG_XD+: no longer U4.C1 (D2+)
- net OTG_XD-: no longer U4.C2 (D2-)
- net VIN_3V3: no longer C12.1, C13.1, R16.1, U5.1 (VCC), U5.20 (VCC), U5.28 (VCC), U5.6 (VCC), U6.10 (VPWER)
- new net HOST_XD+: U4.C1 (D2+)
- new net HOST_XD-: U4.C2 (D2-)
- new net LIVE_3V3: C12.1, C13.1, R16.1, U5.1 (VCC), U5.20 (VCC), U5.28 (VCC), U5.6 (VCC), U6.10 (VPWER)
Changed lines of the file:
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@@
     (effects (font (size 1.27 1.27)) (justify left))
   )
-  (hierarchical_label "VIN_3V3" (shape input) (at 200.66 115.57 0)
+  (hierarchical_label "LIVE_3V3" (shape input) (at 200.66 115.57 0)
     (effects (font (size 1.27 1.27)) (justify left))
   )
-  (hierarchical_label "VIN_3V3" (shape input) (at 200.66 62.23 0)
+  (hierarchical_label "LIVE_3V3" (shape input) (at 200.66 62.23 0)
     (effects (font (size 1.27 1.27)) (justify left))
   )
@@
     (effects (font (size 1.27 1.27)) (justify left))
   )
-  (hierarchical_label "OTG_XD-" (shape input) (at 116.84 36.83 0)
+  (hierarchical_label "HOST_XD-" (shape input) (at 116.84 36.83 0)
     (effects (font (size 1.27 1.27)) (justify left))
   )
@@
     (effects (font (size 1.27 1.27)) (justify right))
   )
-  (hierarchical_label "OTG_XD+" (shape input) (at 116.84 39.37 0)
+  (hierarchical_label "HOST_XD+" (shape input) (at 116.84 39.37 0)
     (effects (font (size 1.27 1.27)) (justify left))
   )
@@
     (effects (font (size 1.27 1.27)) (justify left))
   )
-  (hierarchical_label "VIN_3V3" (shape input) (at 142.24 63.5 0)
+  (hierarchical_label "LIVE_3V3" (shape input) (at 142.24 63.5 0)
     (effects (font (size 1.27 1.27)) (justify left))
   )
