File: Hardware/292/292-power/otg-usb-c.kicad_sch (KiCad schematic)
At the start: 23 parts, among them J5 OTG, U7 TS5USBC410YFFR, U8 TUSB546-DCIRNQT, U9 TPD6S300ARUKR

Commit message: First review based revision
Connections:
- net VIN_3V3 renamed LIVE_3V3
Changed lines of the file:
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@@
     (effects (font (size 1.27 1.27)) (justify left))
   )
-  (hierarchical_label "VIN_3V3" (shape input) (at 203.2 41.91 0)
+  (hierarchical_label "LIVE_3V3" (shape input) (at 203.2 41.91 0)
     (effects (font (size 1.27 1.27)) (justify left))
   )
-  (hierarchical_label "VIN_3V3" (shape input) (at 266.7 127 0)
+  (hierarchical_label "LIVE_3V3" (shape input) (at 266.7 127 0)
     (effects (font (size 1.27 1.27)) (justify left))
   )
@@
     (effects (font (size 1.27 1.27)) (justify left))
   )
-  (hierarchical_label "VIN_3V3" (shape input) (at 55.88 36.83 180)
+  (hierarchical_label "LIVE_3V3" (shape input) (at 55.88 36.83 180)
     (effects (font (size 1.27 1.27)) (justify right))
   )
@@
     (effects (font (size 1.27 1.27)) (justify left))
   )
-  (hierarchical_label "VIN_3V3" (shape input) (at 203.2 95.25 0)
+  (hierarchical_label "LIVE_3V3" (shape input) (at 203.2 95.25 0)
     (effects (font (size 1.27 1.27)) (justify left))
   )
@@
     (effects (font (size 1.27 1.27)) (justify left))
   )
-  (hierarchical_label "VIN_3V3" (shape input) (at 81.28 157.48 0)
+  (hierarchical_label "LIVE_3V3" (shape input) (at 81.28 157.48 0)
     (effects (font (size 1.27 1.27)) (justify left))
   )
@@
     (effects (font (size 1.27 1.27)) (justify left))
   )
-  (hierarchical_label "VIN_3V3" (shape input) (at 154.94 43.18 0)
+  (hierarchical_label "LIVE_3V3" (shape input) (at 154.94 43.18 0)
     (effects (font (size 1.27 1.27)) (justify left))
   )
