File: Hardware/292/292-power/power-part.kicad_sch (KiCad schematic)
At the start: 5 parts

Commit message: Draft board design
Parts:
- added C1, C2, C3, C5: 22uF, Capacitor_SMD:C_0402_1005Metric, symbol Device:C
- added C6: C, Capacitor_SMD:C_0402_1005Metric, symbol Device:C
- added C7: 1uF, Capacitor_SMD:C_0402_1005Metric, symbol Device:C
- added D1, D2: D_Schottky, Diode_SMD:D_0402_1005Metric, symbol Device:D_Schottky
- added L1: L, Inductor_SMD:L_0805_2012Metric, symbol Device:L
- added R2: 47K, Resistor_SMD:R_0402_1005Metric, symbol Device:R
- added R3, R4, R5, R6: R, Resistor_SMD:R_0402_1005Metric, symbol Device:R
- C4: renamed from C?; value C -> 33nF; footprint (none) -> Capacitor_SMD:C_0402_1005Metric
- J1: renamed from J?; value Conn_01x03 -> Lock; footprint (none) -> Connector_JST:JST_ACH_BM03B-ACHSS-GAN-ETF_1x03-1MP_P1.20mm_Vertical
- J2: renamed from J?; value Conn_01x03 -> Battery; footprint (none) -> Connector_JST:JST_ACH_BM03B-ACHSS-GAN-ETF_1x03-1MP_P1.20mm_Vertical
- U2: renamed from U?; footprint RSH0056E -> Ziloo:TPS65988DHRSHR
- U3: renamed from U?; footprint RGE0024H -> Ziloo:BQ24250RGER
Connections:
- net BAT_STAT: now also U3.7 (STAT)
- net POWER_SCL: now also U3.6 (SCL)
- net POWER_SDA: now also U3.5 (SDA)
- net PWR_CHARGE: now also U2.1 (PP_HV2), U2.11 (PP_HV1), U2.12 (PP_HV1), U2.2 (PP_HV2), U3.19 (IN), C1.1
- net LOCK_BTN: now reaches J1.1 (Pin_1)
- net PD_LDO_3V3: now reaches J1.2 (Pin_2)
- net PD_LDO_3V3: now also U2.9 (LDO_3V3)
- net SHUTDOWN_BTN: now reaches J1.3 (Pin_3)
- net OTG_VBUS: now reaches U2.13 (VBUS1)
- net OTG_VBUS: now also U2.14 (VBUS1), D2.1 (K)
- net GND: now reaches U2.15 (DRAIN1)
- net GND: now also J2.3 (Pin_3), U2.19 (DRAIN1), U2.20 (GND), U2.51 (GND), U2.52 (DRAIN2), U2.56 (DRAIN2), U2.57 (DRAIN2), U2.58 (DRAIN1), U2.59 (GND), U2.7 (DRAIN2), U2.8 (DRAIN1), U3.15 (PGND), U3.16 (PGND), U3.25 (PAD), U3.4 (AGND), C1.2, C2.2, C3.2, C5.2, C6.2, C7.2, D1.2 (A), D2.2 (A), R2.2, R3.2, R4.2, R5.2
- net at U2.25 (PP1_CABLE): now also U2.46 (PP2_CABLE), C2.1
- net HOST_VBUS: now reaches U2.3 (VBUS2)
- net HOST_VBUS: now also U2.4 (VBUS2), D1.1 (K)
- net PD_LDO_1V8: now reaches U2.35 (LDO_1V8)
- net BAT_CE_N: now reaches U3.1 (CE_N)
- net BAT_CE_N: now also R2.1
- net at U3.10 (ISET): now also R4.1
- net at U3.11 (BAT): now also J2.1 (Pin_1), U3.12 (BAT), C7.1
- net VSOM: now reaches U3.13 (SYS)
- net VSOM: now also U3.14 (SYS), C5.1, C6.1, L1.2
- net at U3.17 (SW): now also C4.1, U3.18 (SW), L1.1
- net BAT_EN: now reaches U3.2 (EN1)
- net BAT_EN: now also U3.3 (EN2)
- net at U3.21 (BOOT): now also C4.2
- net at U3.22 (ILIM): now also R3.1
- net BAT_LDO: now reaches U3.24 (LDO)
- net BAT_LDO: now also C3.1, R6.2
- net BAT_INT: now reaches U3.8 (INT)
- net at U3.9 (TS): now also J2.2 (Pin_2), R5.1, R6.1
Other:
- note added: "4.9V 50mA"
- note added: "Input from BQ downreg to 3.3V"
- note added: "Input from BQ upreg to 5V"
- note added: "UPREGULATED FROM VSOM"
- note added: "down to 3.0V"
- moved on the sheet: C4, J1, J2, U2B, U3

Commit message: Clarifications for the board plan
Parts:
- added D?: LED, symbol Device:LED
- added R?: R, Resistor_SMD:R_0402_1005Metric, symbol Device:R
- L1: value L -> 1.0uH
Connections:
- net BAT_LDO: now also R?.1
- net BAT_STAT: now also D?.1 (K)
- new net: D?.2 (A), R?.2
Changed lines of the file:
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@@
     (title "Power Charging and Delivery")
   )
+  (junction (at 119.38 50.8) (diameter 0) (color 0 0 0 0)
+  )
   (junction (at 207.01 27.94) (diameter 0) (color 0 0 0 0)
   )
@@
   (junction (at 227.33 64.77) (diameter 0) (color 0 0 0 0)
   )
+  (junction (at 147.32 64.77) (diameter 0) (color 0 0 0 0)
+  )
   (junction (at 96.52 147.32) (diameter 0) (color 0 0 0 0)
   )
@@
     (stroke (width 0) (type default) (color 0 0 0 0))
   )
+  (wire (pts (xy 119.38 67.31) (xy 123.19 67.31))
+    (stroke (width 0) (type default) (color 0 0 0 0))
+  )
   (wire (pts (xy 92.71 165.1) (xy 92.71 166.37))
     (stroke (width 0) (type default) (color 0 0 0 0))
@@
     (stroke (width 0) (type default) (color 0 0 0 0))
   )
+  (wire (pts (xy 119.38 50.8) (xy 119.38 55.88))
+    (stroke (width 0) (type default) (color 0 0 0 0))
+  )
+  (wire (pts (xy 119.38 63.5) (xy 119.38 67.31))
+    (stroke (width 0) (type default) (color 0 0 0 0))
+  )
   (wire (pts (xy 142.24 71.12) (xy 156.21 71.12))
     (stroke (width 0) (type default) (color 0 0 0 0))
@@
     (stroke (width 0) (type default) (color 0 0 0 0))
   )
+  (wire (pts (xy 147.32 64.77) (xy 156.21 64.77))
+    (stroke (width 0) (type default) (color 0 0 0 0))
+  )
   (wire (pts (xy 99.06 149.86) (xy 96.52 149.86))
     (stroke (width 0) (type default) (color 0 0 0 0))
@@
     (stroke (width 0) (type default) (color 0 0 0 0))
   )
+  (wire (pts (xy 147.32 67.31) (xy 147.32 64.77))
+    (stroke (width 0) (type default) (color 0 0 0 0))
+  )
   (wire (pts (xy 196.85 35.56) (xy 199.39 35.56))
     (stroke (width 0) (type default) (color 0 0 0 0))
@@
     (stroke (width 0) (type default) (color 0 0 0 0))
   )
+  (wire (pts (xy 119.38 50.8) (xy 147.32 50.8))
+    (stroke (width 0) (type default) (color 0 0 0 0))
+  )
   (wire (pts (xy 157.48 142.24) (xy 157.48 139.7))
     (stroke (width 0) (type default) (color 0 0 0 0))
@@
     (stroke (width 0) (type default) (color 0 0 0 0))
   )
-  (wire (pts (xy 142.24 50.8) (xy 147.32 50.8))
+  (wire (pts (xy 113.03 50.8) (xy 119.38 50.8))
     (stroke (width 0) (type default) (color 0 0 0 0))
   )
@@
     (stroke (width 0) (type default) (color 0 0 0 0))
   )
-  (wire (pts (xy 142.24 64.77) (xy 156.21 64.77))
+  (wire (pts (xy 144.78 64.77) (xy 147.32 64.77))
     (stroke (width 0) (type default) (color 0 0 0 0))
   )
@@
     (stroke (width 0) (type default) (color 0 0 0 0))
   )
+  (wire (pts (xy 130.81 67.31) (xy 147.32 67.31))
+    (stroke (width 0) (type default) (color 0 0 0 0))
+  )
   (wire (pts (xy 229.87 62.23) (xy 233.68 62.23))
     (stroke (width 0) (type default) (color 0 0 0 0))
@@
     )
   )
-  (text "4.9V 50mA\n" (at 132.08 49.53 0)
+  (text "4.9V 50mA\n" (at 114.3 49.53 0)
     (effects (font (size 1.27 1.27)) (justify left bottom))
   )
@@
     (effects (font (size 1.27 1.27)) (justify left))
   )
-  (hierarchical_label "BAT_LDO" (shape input) (at 142.24 50.8 180)
+  (hierarchical_label "BAT_LDO" (shape input) (at 113.03 50.8 180)
     (effects (font (size 1.27 1.27)) (justify right))
   )
@@
     (effects (font (size 1.27 1.27)) (justify left))
   )
-  (hierarchical_label "BAT_STAT" (shape input) (at 142.24 64.77 180)
+  (hierarchical_label "BAT_STAT" (shape input) (at 144.78 64.77 180)
     (effects (font (size 1.27 1.27)) (justify right))
   )
@@
     (pin "3")
   )
+  (symbol (lib_id "Device:R") (at 119.38 59.69 0) (unit 1)
+    (in_bom yes) (on_board yes)
+    (property "Reference" "R?" (id 0) (at 120.65 55.88 0)
+      (effects (font (size 1.27 1.27)) (justify left))
+    )
+    (property "Value" "R" (id 1) (at 120.65 64.77 0)
+      (effects (font (size 1.27 1.27)) (justify left))
+    )
+    (property "Footprint" "Resistor_SMD:R_0402_1005Metric" (id 2) (at 117.602 59.69 90)
+      (effects (font (size 1.27 1.27)) hide)
+    )
+    (property "Datasheet" "~" (id 3) (at 119.38 59.69 0)
+      (effects (font (size 1.27 1.27)) hide)
+    )
+    (pin "1")
+    (pin "2")
+  )
   (symbol (lib_id "power:GND") (at 227.33 39.37 0) (unit 1)
     (in_bom yes) (on_board yes) (fields_autoplaced)
@@
     (pin "2")
   )
+  (symbol (lib_id "Device:LED") (at 127 67.31 180) (unit 1)
+    (in_bom yes) (on_board yes) (fields_autoplaced)
+    (property "Reference" "D?" (id 0) (at 128.5875 59.69 0))
+    (property "Value" "LED" (id 1) (at 128.5875 62.23 0))
+    (property "Footprint" "" (id 2) (at 127 67.31 0)
+      (effects (font (size 1.27 1.27)) hide)
+    )
+    (property "Datasheet" "~" (id 3) (at 127 67.31 0)
+      (effects (font (size 1.27 1.27)) hide)
+    )
+    (pin "1")
+    (pin "2")
+  )
   (symbol (lib_id "Device:C") (at 207.01 34.29 0) (unit 1)
     (in_bom yes) (on_board yes) (fields_autoplaced)
@@
     (in_bom yes) (on_board yes) (fields_autoplaced)
     (property "Reference" "L1" (id 0) (at 214.63 21.59 90))
-    (property "Value" "L" (id 1) (at 214.63 24.13 90))
+    (property "Value" "1.0uH" (id 1) (at 214.63 24.13 90))
     (property "Footprint" "Inductor_SMD:L_0805_2012Metric" (id 2) (at 214.63 27.94 0)
       (effects (font (size 1.27 1.27)) hide)

Commit message: First review based revision
Parts:
- added C? (x2): C, Capacitor_SMD:C_0402_1005Metric, symbol Device:C
- added C?: 5uF, Capacitor_SMD:C_0402_1005Metric, symbol Device:C
- added U? (x2): TPS79633DCQR, Ziloo:TPS79618DCQR, symbol Ziloo:TPS79618DCQR
Connections:
- net GND: now also U3.23 (VDPM), U?.3 (GND), U?.3 (GND); no longer U2.15 (DRAIN1), U2.19 (DRAIN1), U2.52 (DRAIN2), U2.56 (DRAIN2), U2.57 (DRAIN2), U2.58 (DRAIN1), U2.7 (DRAIN2), U2.8 (DRAIN1)
- net VCC_RTC: now also U2.5 (VIN_3V3), C?.1, U?.4 (OUT)
- net VSOM: now also U?.1 (EN), U?.2 (IN)
- net at C7.1, J2.1 (Pin_1), U3.11 (BAT)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: now also U?.1 (EN), U?.2 (IN)
- new net: C?.1, U?.5 (NR/FB) (x2)
- new net LIVE_3V3: U?.4 (OUT)
- no-connect marks 0 -> 8
Other:
- note removed: "Input from BQ downreg to 3.3V"
- note removed: "down to 3.0V"
- moved on the sheet: C3, C4, C5, C6, C7, D?, J1, J2, L1, R2, R3, R4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
