File: Hardware/929/Faceboard/Faceboard.kicad_sch (KiCad schematic)
At the start: 5 parts, among them P1 UCM-P1, P2 UCM-P2

Commit message: Added components
ESD HDMI
Extra components planned
Parts:
- added U1: SN74CB3Q3245RGYR, Ziloo:SN74CB3Q3245RGYR, symbol Ziloo:SN74CB3Q3245PW
Connections:
- net ?_RXD: now also U1.4 (A3), U1.8 (A7)
- net ?_TXD: now also U1.5 (A4), U1.9 (A8)
- net GND: now also U1.10 (GND)
- net NIGHT_I2C_SCL: now also U1.6 (A5)
- net NIGHT_I2C_SDA: now also U1.7 (A6)
- net SYS_PRG#: now also U1.19 (*OE)
- net F_SBWTCK renamed LEFT_SCL
- net LEFT_SCL: now also U1.2 (A1)
- net F_SBWTDIO renamed LEFT_SDA
- net LEFT_SDA: now also U1.3 (A2)
- new net C_FW_RXD: U1.12 (B7)
- new net C_FW_TXD: U1.11 (B8)
- new net C_SBWTCK: U1.14 (B5)
- new net C_SBWTDIO: U1.13 (B6)
- new net FACE_FW_RXD: U1.16 (B3)
- new net FACE_FW_TXD: U1.15 (B4)
- new net FACE_SBWTCK: U1.18 (B1)
- new net FACE_SBWTDIO: U1.17 (B2)
- new net SLEEP_3V3: U1.20 (VCC)

Commit message: Removed VSOM diodes
Connections:
- net ?_RXD: no longer P1.74 (UART2_TXD), P1.86 (UART4_TXD), U1.4 (A3), U1.8 (A7)
- net ?_TXD: no longer P1.76 (UART2_RXD), P1.84 (UART4_RXD), U1.5 (A4), U1.9 (A8)
- net C_FW_RXD renamed CAM_FW_RXD
- net C_FW_TXD renamed CAM_FW_TXD
- net C_SBWTCK renamed CAM_SBWTCK
- net C_SBWTDIO renamed CAM_SBWTDIO
- new net CORA_TXD: P1.74 (UART2_TXD), U1.4 (A3)
- new net COREA_RXD: P1.76 (UART2_RXD), U1.5 (A4)
- new net COREM_RXD: P1.84 (UART4_RXD), U1.9 (A8)
- new net COREM_TXD: P1.86 (UART4_TXD), U1.8 (A7)
- no-connect marks 18 -> 19

Commit message: PoC board task
Connections:
- net VCC_RTC is gone; now on net SLEEP_3V3: P1.93 (VCC_RTC)
- net CAM_FW_RXD: now also U1.8 (A7); no longer U1.12 (B7)
- net CAM_FW_TXD: now also U1.9 (A8); no longer U1.11 (B8)
- net CAM_SBWTCK: now also U1.6 (A5); no longer U1.14 (B5)
- net CAM_SBWTDIO: now also U1.7 (A6); no longer U1.13 (B6)
- net COREA_RXD: now also P1.74 (UART2_TXD), U1.16 (B3); no longer P1.76 (UART2_RXD), U1.5 (A4)
- net COREM_RXD: now also P1.86 (UART4_TXD), U1.12 (B7); no longer P1.84 (UART4_RXD), U1.9 (A8)
- net COREM_TXD: now also P1.84 (UART4_RXD), U1.11 (B8); no longer P1.86 (UART4_TXD), U1.8 (A7)
- net FACE_FW_RXD: now also U1.4 (A3); no longer U1.16 (B3)
- net FACE_FW_TXD: now also U1.5 (A4); no longer U1.15 (B4)
- net FACE_SBWTCK: now also U1.2 (A1); no longer U1.18 (B1)
- net FACE_SBWTDIO: now also U1.3 (A2); no longer U1.17 (B2)
- net NIGHT_I2C_SCL: now also U1.14 (B5); no longer U1.6 (A5)
- net NIGHT_I2C_SDA: now also U1.13 (B6); no longer U1.7 (A6)
- net CAN2_RX: now reaches P1.49 (CAN2_RX)
- net +VDC renamed VSOM
- net ?_RXD renamed STEM_MSG_TXD
- net STEM_MSG_TXD: no longer P1.61 (UART3_TXD)
- net ?_TXD renamed STEM_MSG_RXD
- net STEM_MSG_RXD: no longer P1.21 (UART3_RXD)
- removed net CORA_TXD: P1.74 (UART2_TXD), U1.4 (A3)
- net LEFT_SCL renamed DAY_I2C_SCL
- net DAY_I2C_SCL: now also U1.18 (B1); no longer U1.2 (A1)
- net LEFT_SDA renamed DAY_I2C_SDA
- net DAY_I2C_SDA: now also U1.17 (B2); no longer U1.3 (A2)
- net SAI5_RX_DATA1 renamed SAI5_RXD1
- net SAI5_RX_DATA2 renamed SAI5_RXD2
- net SAI5_RX_SYNC renamed SAI5_RXFS
- net STEM_INT renamed GPIO1_IO1
- new net COREA_TXD: P1.76 (UART2_RXD), U1.15 (B4)
- new net UART3_RXD: P1.21 (UART3_RXD)
- new net UART3_TXD: P1.61 (UART3_TXD)
Other:
- moved on the sheet: C100, C101, C102, U1
