File: Hardware/929/Faceboard/ethernet-sd1.kicad_sch (KiCad schematic)
At the start: 16 parts, among them J2 Raspberry_Pi_to_Ziloo, J4 RJ45

Commit message: PoC board task
Parts:
- added J5: UCM-P20-misc, Connector_PinHeader_2.54mm:PinHeader_2x17_P2.54mm_Vertical_SMD, symbol Ziloo:UCM-P20-misc
- added J6: UCM-P21-misc, Connector_PinHeader_2.54mm:PinHeader_2x17_P2.54mm_Vertical_SMD, symbol Ziloo:UCM-P21-misc
- added P4: Power, Connector_PinHeader_2.54mm:PinHeader_2x06_P2.54mm_Vertical_SMD, symbol Connector_Generic:Conn_02x06_Odd_Even
- gave numbers to parts that had none: 1
Connections:
- net GND: now also J5.31 (GND), J5.32 (GND), J6.6 (GND), J6.9 (GND), P4.11 (Pin_11), P4.12 (Pin_12)
- net HDMI_5V: now also P4.1 (Pin_1), P4.7 (Pin_7); no longer J2.2 (5V), J2.4 (5V)
- net LIVE_3V3: now also P4.3 (Pin_3), P4.9 (Pin_9); no longer J2.1 (3V3), J2.17 (3V3)
- net MCU_SYS_INT: now also J5.20 (MCU_SYS_INT)
- net SAI5_RXD2: now also J6.13 (SAI5_RX_DATA2)
- net SD1_CLK: now also J5.15 (SD1_CLK)
- net SD1_CMD: now also J5.17 (SD1_CMD)
- net SD1_DATA0: now also J5.24 (SD1_DATA0)
- net SD1_DATA1: now also J5.22 (SD1_DATA1)
- net SD1_DATA2: now also J5.21 (SD1_DATA2)
- net SD1_DATA3: now also J5.23 (SD1_DATA3)
- net SD1_RESET_B: now also J5.13 (SD1_RESET_B)
- net STEM_I2C_SCL: now also J5.33 (STEM_SCL)
- net STEM_I2C_SDA: now also J5.34 (STEM_SDA)
- net SYS_I2C_SCL: now also J6.7 (SYS_I2C_SCL)
- net SYS_I2C_SDA: now also J6.5 (SYS_I2C_SDA)
- net SYS_PRG#: now also J5.30 (SYS_PRG)
- new net COEX: J5.18 (COEX)
- new net COREA_RXD: J5.1 (CONSOLE_RXD)
- new net COREA_TXD: J5.3 (CONSOLE_TXD)
- new net COREM_RXD: J5.8 (M7_CON_RXD)
- new net COREM_TXD: J5.10 (M7_CON_TXD)
- new net DAY_I2C_SCL: J6.3 (I2C5_SCL)
- new net DAY_I2C_SDA: J6.1 (I2C5_SDA)
- new net GPIO1_IO1: J5.14 (GPIO1_01)
- new net NIGHT_I2C_SCL: J6.2 (I2C6_SCL)
- new net NIGHT_I2C_SDA: J6.4 (I2C6_SDA)
- new net OE_CAM: J5.27 (OE_CAM)
- new net OE_SOUND: J5.25 (OE_SOUND)
- new net RPI_3V3: J2.1 (3V3), J2.17 (3V3), P4.10 (Pin_10)
- new net RPI_5V: J2.2 (5V), J2.4 (5V), P4.8 (Pin_8)
- new net SAI5_RXC: J6.19 (SAI5_RXC)
- new net SAI5_RXD1: J6.21 (SAI5_RX_DATA1)
- new net SAI5_RXFS: J6.23 (SAI5_RX_SYNC)
- new net SD2_nRST: J6.16 (GPIO2_IO19)
- new net SOUND_INT: J5.12 (SOUND_INT)
- new net STEM_MSG_RXD: J5.11 (STEM_MSG_RXD)
- new net STEM_MSG_TXD: J5.9 (STEM_MSG_TXD)
- new net UART3_RXD: J5.4 (UART3_RXD)
- new net UART3_TXD: J5.2 (UART3_TXD)
- new net UCM_3V3: J5.7 (3V3), P4.4 (Pin_4)
- new net UCM_5V: J5.6 (5V0), P4.2 (Pin_2)
- no-connect marks 0 -> 13
Other:
- note added: "TODO power headers to enable/disable 3V3 5V"
- moved on the sheet: D11, D18, D19, J4, R1, R2, U23
